File: hardware/KiCad Files/LoFi_Oscillator/LoFi_Oscillator.kicad_sch (KiCad schematic)
At the start: 17 parts

Commit message: Initial firmware sketch
Includes Teensy Audio library sketch
Parts:
- renumbered Wavefold to Wavefold2
Other:
- moved on the sheet: AudioOut1, LFOout1
Changed lines of the file:
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@@
     )
   )
-  (symbol (lib_id "eurocad:PJ301M-12") (at 259.08 133.35 180) (unit 1)
-    (in_bom yes) (on_board yes) (dnp no) (fields_autoplaced)
-    (property "Reference" "LFOout1" (at 271.78 131.445 0)
-      (effects (font (size 1.27 1.27)) (justify right))
-    )
-    (property "Value" "PJ301M-12" (at 271.78 133.985 0)
-      (effects (font (size 1.27 1.27)) (justify right))
-    )
-    (property "Footprint" "Thonkiconn:PJ301M-12" (at 271.78 136.525 0)
-      (effects (font (size 1.27 1.27)) (justify right))
-    )
-    (property "Datasheet" "" (at 259.08 133.35 0)
+  (symbol (lib_id "eurocad:PJ301M-12") (at 223.52 115.57 180) (unit 1)
+    (in_bom yes) (on_board yes) (dnp no) (fields_autoplaced)
+    (property "Reference" "LFOout1" (at 236.22 113.665 0)
+      (effects (font (size 1.27 1.27)) (justify right))
+    )
+    (property "Value" "PJ301M-12" (at 236.22 116.205 0)
+      (effects (font (size 1.27 1.27)) (justify right))
+    )
+    (property "Footprint" "Thonkiconn:PJ301M-12" (at 236.22 118.745 0)
+      (effects (font (size 1.27 1.27)) (justify right))
+    )
+    (property "Datasheet" "" (at 223.52 115.57 0)
       (effects (font (size 1.27 1.27)))
     )
@@
     )
   )
-  (symbol (lib_id "eurocad:PJ301M-12") (at 259.08 149.86 180) (unit 1)
-    (in_bom yes) (on_board yes) (dnp no) (fields_autoplaced)
-    (property "Reference" "AudioOut1" (at 271.78 147.955 0)
-      (effects (font (size 1.27 1.27)) (justify right))
-    )
-    (property "Value" "PJ301M-12" (at 271.78 150.495 0)
-      (effects (font (size 1.27 1.27)) (justify right))
-    )
-    (property "Footprint" "Thonkiconn:PJ301M-12" (at 271.78 153.035 0)
-      (effects (font (size 1.27 1.27)) (justify right))
-    )
-    (property "Datasheet" "" (at 259.08 149.86 0)
+  (symbol (lib_id "eurocad:PJ301M-12") (at 223.52 132.08 180) (unit 1)
+    (in_bom yes) (on_board yes) (dnp no) (fields_autoplaced)
+    (property "Reference" "AudioOut1" (at 236.22 130.175 0)
+      (effects (font (size 1.27 1.27)) (justify right))
+    )
+    (property "Value" "PJ301M-12" (at 236.22 132.715 0)
+      (effects (font (size 1.27 1.27)) (justify right))
+    )
+    (property "Footprint" "Thonkiconn:PJ301M-12" (at 236.22 135.255 0)
+      (effects (font (size 1.27 1.27)) (justify right))
+    )
+    (property "Datasheet" "" (at 223.52 132.08 0)
       (effects (font (size 1.27 1.27)))
     )
@@
   (symbol (lib_id "eurocad:PJ301M-12") (at 25.4 102.87 0) (unit 1)
     (in_bom yes) (on_board yes) (dnp no) (fields_autoplaced)
-    (property "Reference" "Wavefold" (at 23.495 90.17 0)
+    (property "Reference" "Wavefold2" (at 23.495 90.17 0)
       (effects (font (size 1.27 1.27)))
     )
@@
       (project "LoFi_Oscillator"
         (path "/f59f5373-0fe4-4ba6-a94e-273ab7a336aa"
-          (reference "Wavefold") (unit 1)
-        )
-      )
+          (reference "Wavefold2") (unit 1)
+        )
+      )
